File: hardware/eprom27_programmer.kicad_sch (KiCad schematic)
At the start: 43 parts, among them IC1 EPROM, J1 Prog DC In, J2 Prog DC In, M1 MT3608, Q1 BC547, Q10 BC557, Q2 BC557, Q3 BC547, Q4 BC557, Q5 BC547, Q6 BC557, Q7 BC557, Q8 BC557, Q9 BC547, U1 74HC595, U2 74HC595

Commit message: Change voltage naming Update voltage divider Update README
Signed-off-by: Ilias Daradimos <judgedrid@gmail.com>
Parts:
- R1: value 10k -> 33k
- R2: value 15k -> 6.8k
Connections:
- net +24V renamed VPP
- net VCC renamed +5V
Changed lines of the file:
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@@
     (rev "${revision}")
     (comment 1 "${comment1}")
-    (comment 2 "${description}")
   )
   (junction (at 90.805 145.415) (diameter 0) (color 0 0 0 0)
@@
     )
   )
-  (symbol (lib_id "power:+24V") (at 106.045 130.81 0) (unit 1)
+  (symbol (lib_id "power:VPP") (at 106.045 130.81 0) (unit 1)
     (in_bom yes) (on_board yes) (dnp no) (fields_autoplaced)
     (property "Reference" "#P+03" (at 106.045 130.81 0)
       (effects (font (size 1.27 1.27)) hide)
     )
-    (property "Value" "+24V" (at 106.045 126.365 0)
-      (effects (font (size 1.778 1.5113)))
+    (property "Value" "VPP" (at 107.95 129.54 0)
+      (effects (font (size 1.778 1.5113)) (justify left))
     )
     (property "Footprint" "" (at 106.045 130.81 0)
@@
     )
   )
-  (symbol (lib_id "power:+24V") (at 245.11 143.51 0) (unit 1)
+  (symbol (lib_id "power:VPP") (at 245.11 143.51 0) (unit 1)
     (in_bom yes) (on_board yes) (dnp no) (fields_autoplaced)
     (property "Reference" "#P+07" (at 245.11 143.51 0)
       (effects (font (size 1.27 1.27)) hide)
     )
-    (property "Value" "+24V" (at 243.205 142.24 0)
-      (effects (font (size 1.778 1.5113)) (justify right))
+    (property "Value" "VPP" (at 247.65 142.24 0)
+      (effects (font (size 1.778 1.5113)) (justify left))
     )
     (property "Footprint" "" (at 245.11 143.51 0)
@@
     )
   )
-  (symbol (lib_id "power:VCC") (at 131.445 24.765 0) (unit 1)
+  (symbol (lib_id "power:+5V") (at 131.445 24.765 0) (unit 1)
     (in_bom yes) (on_board yes) (dnp no) (fields_autoplaced)
     (property "Reference" "#PWR05" (at 131.445 28.575 0)
       (effects (font (size 1.27 1.27)) hide)
     )
-    (property "Value" "VCC" (at 131.445 20.955 0)
+    (property "Value" "+5V" (at 131.445 20.32 0)
       (effects (font (size 1.27 1.27)))
     )
@@
     )
   )
-  (symbol (lib_id "power:+24V") (at 262.89 114.3 0) (unit 1)
+  (symbol (lib_id "power:VPP") (at 262.89 114.3 0) (unit 1)
     (in_bom yes) (on_board yes) (dnp no) (fields_autoplaced)
     (property "Reference" "#P+08" (at 262.89 114.3 0)
       (effects (font (size 1.27 1.27)) hide)
     )
-    (property "Value" "+24V" (at 262.89 109.855 0)
-      (effects (font (size 1.778 1.5113)))
+    (property "Value" "VPP" (at 265.43 113.03 0)
+      (effects (font (size 1.778 1.5113)) (justify left))
     )
     (property "Footprint" "" (at 262.89 114.3 0)
@@
     )
   )
-  (symbol (lib_id "power:VCC") (at 130.175 82.55 0) (unit 1)
-    (in_bom yes) (on_board yes) (dnp no) (fields_autoplaced)
+  (symbol (lib_id "power:+5V") (at 130.175 82.55 0) (unit 1)
+    (in_bom yes) (on_board yes) (dnp no)
     (property "Reference" "#PWR03" (at 130.175 86.36 0)
       (effects (font (size 1.27 1.27)) hide)
     )
-    (property "Value" "VCC" (at 130.175 78.74 0)
+    (property "Value" "+5V" (at 128.27 78.74 0)
       (effects (font (size 1.27 1.27)))
     )
@@
     )
   )
-  (symbol (lib_id "power:VCC") (at 151.765 132.715 0) (unit 1)
+  (symbol (lib_id "power:+5V") (at 151.765 132.715 0) (unit 1)
     (in_bom yes) (on_board yes) (dnp no) (fields_autoplaced)
     (property "Reference" "#P+05" (at 151.765 132.715 0)
       (effects (font (size 1.27 1.27)) hide)
     )
-    (property "Value" "VCC" (at 151.765 127.635 0)
+    (property "Value" "+5V" (at 151.765 127 0)
       (effects (font (size 1.778 1.5113)))
     )
@@
     )
   )
-  (symbol (lib_id "power:VCC") (at 192.405 24.765 0) (unit 1)
+  (symbol (lib_id "power:+5V") (at 192.405 24.765 0) (unit 1)
     (in_bom yes) (on_board yes) (dnp no) (fields_autoplaced)
     (property "Reference" "#PWR07" (at 192.405 28.575 0)
       (effects (font (size 1.27 1.27)) hide)
     )
-    (property "Value" "VCC" (at 192.405 20.955 0)
+    (property "Value" "+5V" (at 192.405 20.32 0)
       (effects (font (size 1.27 1.27)))
     )
@@
     )
   )
-  (symbol (lib_id "power:VCC") (at 265.43 143.51 0) (unit 1)
+  (symbol (lib_id "power:+5V") (at 265.43 143.51 0) (unit 1)
     (in_bom yes) (on_board yes) (dnp no) (fields_autoplaced)
     (property "Reference" "#P+09" (at 265.43 143.51 0)
       (effects (font (size 1.27 1.27)) hide)
     )
-    (property "Value" "VCC" (at 267.335 142.24 0)
+    (property "Value" "+5V" (at 267.97 142.24 0)
       (effects (font (size 1.778 1.5113)) (justify left))
     )
@@
     )
   )
-  (symbol (lib_id "power:VCC") (at 73.66 41.275 0) (unit 1)
+  (symbol (lib_id "power:+5V") (at 73.66 41.275 0) (unit 1)
     (in_bom yes) (on_board yes) (dnp no) (fields_autoplaced)
     (property "Reference" "#PWR02" (at 73.66 45.085 0)
       (effects (font (size 1.27 1.27)) hide)
     )
-    (property "Value" "VCC" (at 73.66 37.465 0)
+    (property "Value" "+5V" (at 73.66 36.83 0)
       (effects (font (size 1.27 1.27)))
     )
@@
     )
   )
-  (symbol (lib_id "power:VCC") (at 164.465 132.715 0) (unit 1)
+  (symbol (lib_id "power:+5V") (at 164.465 132.715 0) (unit 1)
     (in_bom yes) (on_board yes) (dnp no) (fields_autoplaced)
     (property "Reference" "#P+06" (at 164.465 132.715 0)
       (effects (font (size 1.27 1.27)) hide)
     )
-    (property "Value" "VCC" (at 164.465 127.635 0)
-      (effects (font (size 1.778 1.5113)))
+    (property "Value" "+5V" (at 166.37 131.445 0)
+      (effects (font (size 1.778 1.5113)) (justify left))
     )
     (property "Footprint" "" (at 164.465 132.715 0)
@@
     )
   )
-  (symbol (lib_id "power:+24V") (at 136.525 130.81 0) (unit 1)
+  (symbol (lib_id "power:VPP") (at 136.525 130.81 0) (unit 1)
     (in_bom yes) (on_board yes) (dnp no) (fields_autoplaced)
     (property "Reference" "#P+04" (at 136.525 130.81 0)
       (effects (font (size 1.27 1.27)) hide)
     )
-    (property "Value" "+24V" (at 136.525 126.365 0)
-      (effects (font (size 1.778 1.5113)))
+    (property "Value" "VPP" (at 138.43 129.54 0)
+      (effects (font (size 1.778 1.5113)) (justify left))
     )
     (property "Footprint" "" (at 136.525 130.81 0)
@@
   (symbol (lib_id "Device:R") (at 97.155 34.925 0) (unit 1)
     (in_bom yes) (on_board yes) (dnp no) (fields_autoplaced)
-    (property "Reference" "R1" (at 94.615 33.655 0)
+    (property "Reference" "R1" (at 95.25 33.02 0)
       (effects (font (size 1.778 1.5113)) (justify right))
     )
-    (property "Value" "10k" (at 94.615 36.195 0)
+    (property "Value" "33k" (at 95.25 36.83 0)
       (effects (font (size 1.778 1.5113)) (justify right))
     )
@@
     )
   )
-  (symbol (lib_id "power:+24V") (at 75.565 130.81 0) (unit 1)
+  (symbol (lib_id "power:VPP") (at 75.565 130.81 0) (unit 1)
     (in_bom yes) (on_board yes) (dnp no) (fields_autoplaced)
     (property "Reference" "#P+01" (at 75.565 130.81 0)
       (effects (font (size 1.27 1.27)) hide)
     )
-    (property "Value" "+24V" (at 75.565 126.365 0)
-      (effects (font (size 1.778 1.5113)))
+    (property "Value" "VPP" (at 77.47 129.54 0)
+      (effects (font (size 1.778 1.5113)) (justify left))
     )
     (property "Footprint" "" (at 75.565 130.81 0)
@@
     )
   )
-  (symbol (lib_id "power:+24V") (at 97.155 29.845 0) (unit 1)
+  (symbol (lib_id "power:VPP") (at 97.155 29.845 0) (unit 1)
     (in_bom yes) (on_board yes) (dnp no) (fields_autoplaced)
     (property "Reference" "#P+02" (at 97.155 29.845 0)
       (effects (font (size 1.27 1.27)) hide)
     )
-    (property "Value" "+24V" (at 94.615 29.5275 0)
+    (property "Value" "VPP" (at 99.06 28.575 0)
+      (effects (font (size 1.778 1.5113)) (justify left))
+    )
+    (property "Footprint" "" (at 97.155 29.845 0)
+      (effects (font (size 1.27 1.27)) hide)
+    )
+    (property "Datasheet" "" (at 97.155 29.845 0)
+      (effects (font (size 1.27 1.27)) hide)
+    )
+    (pin "1")
+    (instances
+      (project "eprom27_programmer"
+        (path "/111a49a6-2ada-45ca-8c70-190362b471de"
+          (reference "#P+02") (unit 1)
+        )
+      )
+    )
+  )
+  (symbol (lib_id "Device:R") (at 97.155 48.895 0) (unit 1)
+    (in_bom yes) (on_board yes) (dnp no) (fields_autoplaced)
+    (property "Reference" "R2" (at 95.25 46.99 0)
       (effects (font (size 1.778 1.5113)) (justify right))
     )
-    (property "Footprint" "" (at 97.155 29.845 0)
-      (effects (font (size 1.27 1.27)) hide)
-    )
-    (property "Datasheet" "" (at 97.155 29.845 0)
-      (effects (font (size 1.27 1.27)) hide)
-    )
-    (pin "1")
-    (instances
-      (project "eprom27_programmer"
-        (path "/111a49a6-2ada-45ca-8c70-190362b471de"
-          (reference "#P+02") (unit 1)
-        )
-      )
-    )
-  )
-  (symbol (lib_id "Device:R") (at 97.155 48.895 0) (unit 1)
-    (in_bom yes) (on_board yes) (dnp no) (fields_autoplaced)
-    (property "Reference" "R2" (at 94.615 47.625 0)
-      (effects (font (size 1.778 1.5113)) (justify right))
-    )
-    (property "Value" "15k" (at 94.615 50.165 0)
+    (property "Value" "6.8k" (at 95.25 50.8 0)
       (effects (font (size 1.778 1.5113)) (justify right))
     )
@@
     )
   )
-  (symbol (lib_id "power:+24V") (at 41.275 130.81 0) (unit 1)
+  (symbol (lib_id "power:VPP") (at 41.275 130.81 0) (unit 1)
     (in_bom yes) (on_board yes) (dnp no) (fields_autoplaced)
     (property "Reference" "#P+010" (at 41.275 130.81 0)
       (effects (font (size 1.27 1.27)) hide)
     )
-    (property "Value" "+24V" (at 41.275 126.365 0)
-      (effects (font (size 1.778 1.5113)))
+    (property "Value" "VPP" (at 43.18 129.54 0)
+      (effects (font (size 1.778 1.5113)) (justify left))
     )
     (property "Footprint" "" (at 41.275 130.81 0)
